File: 4_KiCAD_Files/BEEFBoard/BEEFBoard.kicad_sch (KiCad schematic)
At the start: 111 parts, among them J1 Screw_Terminal_01x03, J2 Screw_Terminal_01x03, J3 USB_B_Micro, SW1 SW_MEC_5E, SW10 SW_SPST, SW11 SW_Slide_DPDT, SW12 SW_Slide_DPDT, SW2 SW_SPDT_321, SW3 SW_SPST, SW4 SW_SPST, SW5 SW_SPST, SW6 SW_SPST, SW7 SW_SPST, SW8 SW_SPST, SW9 SW_SPST, U1 STM32H753ZITx, U10 TCAN332G, U11 TCAN332G, U12 LAN8742A, U13 USBLC6-4SC6, U14 USBLC6-2SC6, U2 TQL851CSV33_RLG, U3 INA228, U4 INA228, U5 INA228, U6 INA228, U7 LM317HV_TO-220, U8 LM317HV_TO-220, U9 LM317HV_TO-220, Y1 25MHz, Y2 Crystal_Small

Commit message: Started to work on e-fuses
Parts:
- removed C19: 10u, symbol Device:C_Small
- removed C20: 100n, symbol Device:C_Small
- removed J1, J2: Screw_Terminal_01x03, symbol Connector:Screw_Terminal_01x03
- removed SW10, SW3, SW4, SW5, SW6, SW7, SW8, SW9: SW_SPST, symbol Switch:SW_SPST
- removed U2: TQL851CSV33_RLG, TQL851CSV33_RLG:VREG_TQL851CSV33_RLG, symbol TQL851CSV33_RLG:TQL851CSV33_RLG
- added D7: LED_Small, symbol Device:LED_Small
- added J4, J5: Conn_01x03_Pin, symbol Connector:Conn_01x03_Pin
- added R19: 1k, symbol Device:R_Small
- added R20: 3.6k, symbol Device:R_Small
- added R25: 970k, symbol Device:R_Small
- added R26: 6k, symbol Device:R_Small
- added R45: 24k, symbol Device:R_Small
- added SW13, SW14, SW15, SW16: SW_DIP_x02, Button_Switch_THT:SW_DIP_SPSTx02_Slide_9.78x7.26mm_W7.62mm_P2.54mm, symbol Switch:SW_DIP_x02
- added U15: AZ1084-3.3, symbol Regulator_Linear:AZ1084-3.3
- added U16, U17, U18: TPS25940ARVCR, RVC0020A, symbol TPS25940ARVCR:TPS25940ARVCR
- added U2: TPS26631PWP, Package_SO:HTSSOP-20-1EP_4.4x6.5mm_P0.65mm_EP3.4x6.5mm_Mask2.96x2.96mm_ThermalVias, symbol Power_Management:TPS26631PWP
- C18: value 100n -> 22u
- U10, U11: footprint (none) -> Package_SO:JEITA_SOIC-8_3.9x4.9mm_P1.27mm
Connections:
- net +12VBus: now also U16.4 (OUT), U16.5 (OUT), U16.6 (OUT), U16.7 (OUT), U16.8 (OUT); no longer D3.2 (A), R37.2, U4.9 (Vin-)
- net +3.3V: now also D7.2 (A), U15.2 (VO)
- net +3.3VBus: now also U18.4 (OUT), U18.5 (OUT), U18.6 (OUT), U18.7 (OUT), U18.8 (OUT); no longer D5.2 (A), R39.2, U6.9 (Vin-)
- net +5VBus: now also U17.4 (OUT), U17.5 (OUT), U17.6 (OUT), U17.7 (OUT), U17.8 (OUT); no longer D4.2 (A), R38.2, U5.9 (Vin-)
- net GND: now also J4.2 (Pin_2), J5.2 (Pin_2), R19.2, R20.2, R45.2, U15.1 (GND), U16.16 (GND), U16.21 (PAD), U17.16 (GND), U17.21 (PAD), U18.16 (GND), U18.21 (PAD), U2.21 (GND), U2.9 (GND)
- net I2C_SCL: now also SW13.3, SW14.3, SW15.3, SW16.3
- net I2C_SDA: now also SW13.4, SW14.4, SW15.4, SW16.4
- net at R15.1, R17.1, U4.4 (SDA): now also SW14.1
- net at R10.1, R8.1, U3.5 (SCL): now also SW13.2
- net at R22.1, R24.1, U5.5 (SCL): now also SW15.2
- net at R28.1, R30.1, U6.2 (A0)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: now also SW16.2
- net at SW12.4 (A), U10.6 (CANL): now also J4.1 (Pin_1)
- net at SW12.1 (A), U10.7 (CANH): now also J4.3 (Pin_3)
- net at R21.1, R23.1, U5.2 (A0)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: now also SW15.1
- net at R16.1, R18.1, U4.5 (SCL): now also SW14.2
- net at SW11.4 (A), U11.6 (CANL): now also J5.1 (Pin_1)
- net at SW11.1 (A), U11.7 (CANH): now also J5.3 (Pin_3)
- net at R27.1, R29.1, U6.4 (SDA): now also SW16.1
- net at R7.1, R9.1, U3.4 (SDA): now also SW13.1
- net +12V renamed +12VBATT
- net +12VBATT: now also U15.3 (VI)
- net +BATT renamed +48VBATT
- net +BATTBus renamed +48VBus
- net +48VBus: now also U2.18 (OUT), U2.19 (OUT), U2.20 (OUT); no longer D6.2 (A), R40.2, U3.9 (Vin-)
- new net: D4.2 (A), R38.2, U17.10 (IN), U17.11 (IN), U17.12 (IN), U17.13 (IN), U17.9 (IN), U5.9 (Vin-)
- new net: D7.1 (K), R19.1
- new net: D3.2 (A), R37.2, U16.10 (IN), U16.11 (IN), U16.12 (IN), U16.13 (IN), U16.9 (IN), U4.9 (Vin-)
- new net: D6.2 (A), R25.1, R40.2, U2.1 (IN), U2.2 (IN), U2.3 (IN), U2.6 (IN_SYS), U3.9 (Vin-)
- new net: R25.2, R26.1, U2.7 (UVLO)
- new net: R20.1, U2.11 (ILIM)
- new net: R26.2, R45.1, U2.8 (OVP)
- new net: D5.2 (A), R39.2, U18.10 (IN), U18.11 (IN), U18.12 (IN), U18.13 (IN), U18.9 (IN), U6.9 (Vin-)
- no-connect marks 6 -> 9
Other:
- note added: "1.2V"
- note added: "Might need RCB and RPP here?"
- note added: "Need headers as well probably"
- note added: "The resistor may need work to find the closest standard values"
- note added: "This LED/resistor needs to either be isolated or rated to the high voltage of the battery or isolate it using a pmos or something but then the pmos will have to be rated properly"
- note removed: "This LED/resistor needs to either be isolated or rated to the high voltage of the battery"
- note removed: "might want to reevaluate this part - ask carlo"
- moved on the sheet: C18, C21, C22, C23, C24, C25, C26, C27, C28, C29, D3, D4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
