File: 4_KiCAD_Files/BEEFBoard/BEEFBoard.kicad_sch (KiCad schematic)
At the start: 115 parts, among them J3 USB_B_Micro, J4 Conn_01x03_Pin, J5 Conn_01x03_Pin, SW1 SW_MEC_5E, SW11 SW_Slide_DPDT, SW12 SW_Slide_DPDT, SW13 SW_DIP_x02, SW14 SW_DIP_x02, SW15 SW_DIP_x02, SW16 SW_DIP_x02, SW2 SW_SPDT_321, U1 STM32H753ZITx, U10 TCAN332G, U11 TCAN332G, U12 LAN8742A, U13 USBLC6-4SC6, U14 USBLC6-2SC6, U15 AZ1084-3.3, U16 TPS25940ARVCR, U17 TPS25940ARVCR, U18 TPS25940ARVCR, U2 TPS26631PWP, U3 INA228, U4 INA228, U5 INA228, U6 INA228, U7 LM317HV_TO-220, U8 LM317HV_TO-220, U9 LM317HV_TO-220, Y1 25MHz, Y2 Crystal_Small

Commit message: pushing everzthing iäve done so far before laptop needs to be repaired
Parts:
- added C19, C20: 1u, symbol Device:C_Small
- added J1, J2, J6, J7: Screw_Terminal_01x02, symbol Connector:Screw_Terminal_01x02
- added R46: 249k, symbol Device:R_Small
- added R47: 10k, symbol Device:R_Small
- R26: value 6k -> 6.04k
Connections:
- net +12VBus: now also J1.1 (Pin_1)
- net +3.3VBus: now also J6.1 (Pin_1)
- net +48VBus: now also C19.1, J7.1 (Pin_1), R46.1
- net +5VBus: now also J2.1 (Pin_1)
- net GND: now also C19.2, C20.2, J1.2 (Pin_2), J2.2 (Pin_2), J6.2 (Pin_2), J7.2 (Pin_2), R47.2
- net at D6.2 (A), R25.1, R40.2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: now also C20.1
- net at U2.16 (PGTH): now also R46.2, R47.1
- no-connect marks 9 -> 11
Other:
- note added: "We want heatsinks on these convertors"
- note removed: "1.2V"
- note removed: "The resistor may need work to find the closest standard values"
- moved on the sheet: C18, C21, D7, R19, U15
